File: KiCAD/ExperimentNAND/ExperimentNAND.kicad_sch (KiCad schematic)
At the start: 6 parts, among them U1 MCP4801, U2 MCP4801, U3 ADS1115IDGS, U4 ESP32-DevKitC, U5 74HC00, U6 74HC00

Commit message: updated kicad
Parts:
- added J1: VCC, symbol Connector:Conn_01x03_Pin
Connections:
- net +5V: now also J1.1 (Pin_1); no longer U6.14 (VCC)
- new net: J1.2 (Pin_2), U6.14 (VCC)
- new net +3.3V: J1.3 (Pin_3)
Changed lines of the file:
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@@
+    (stroke (width 0) (type default))
+  )
+  (wire (pts (xy 265.43 31.75) (xy 265.43 29.21))
     (stroke (width 0) (type default))
   )
@@
     (stroke (width 0) (type default))
   )
+  (wire (pts (xy 270.51 31.75) (xy 265.43 31.75))
+    (stroke (width 0) (type default))
+  )
   (wire (pts (xy 217.17 30.48) (xy 237.49 30.48))
     (stroke (width 0) (type default))
@@
     (stroke (width 0) (type default))
   )
+  (wire (pts (xy 270.51 27.94) (xy 270.51 31.75))
+    (stroke (width 0) (type default))
+  )
   (wire (pts (xy 91.44 97.79) (xy 107.95 97.79))
     (stroke (width 0) (type default))
@@
     (stroke (width 0) (type default))
   )
+  (wire (pts (xy 262.89 29.21) (xy 262.89 36.83))
+    (stroke (width 0) (type default))
+  )
+  (wire (pts (xy 255.27 31.75) (xy 260.35 31.75))
+    (stroke (width 0) (type default))
+  )
   (wire (pts (xy 194.31 92.71) (xy 194.31 104.14))
     (stroke (width 0) (type default))
@@
     (stroke (width 0) (type default))
   )
+  (wire (pts (xy 260.35 31.75) (xy 260.35 29.21))
+    (stroke (width 0) (type default))
+  )
   (wire (pts (xy 194.31 87.63) (xy 196.85 87.63))
     (stroke (width 0) (type default))
@@
   )
   (wire (pts (xy 143.51 86.36) (xy 148.59 86.36))
+    (stroke (width 0) (type default))
+  )
+  (wire (pts (xy 255.27 27.94) (xy 255.27 31.75))
     (stroke (width 0) (type default))
   )
@@
     (effects (font (size 1.27 1.27)) (justify right bottom))
   )
-  (symbol (lib_id "power:+5V") (at 262.89 36.83 0) (unit 1)
-    (in_bom yes) (on_board yes) (dnp no) (fields_autoplaced)
-    (property "Reference" "#PWR014" (at 262.89 40.64 0)
-      (effects (font (size 1.27 1.27)) hide)
-    )
-    (property "Value" "+5V" (at 262.89 31.75 0)
-      (effects (font (size 1.27 1.27)))
-    )
-    (property "Footprint" "" (at 262.89 36.83 0)
-      (effects (font (size 1.27 1.27)) hide)
-    )
-    (property "Datasheet" "" (at 262.89 36.83 0)
+  (symbol (lib_id "power:+5V") (at 270.51 27.94 0) (unit 1)
+    (in_bom yes) (on_board yes) (dnp no) (fields_autoplaced)
+    (property "Reference" "#PWR014" (at 270.51 31.75 0)
+      (effects (font (size 1.27 1.27)) hide)
+    )
+    (property "Value" "+5V" (at 270.51 22.86 0)
+      (effects (font (size 1.27 1.27)))
+    )
+    (property "Footprint" "" (at 270.51 27.94 0)
+      (effects (font (size 1.27 1.27)) hide)
+    )
+    (property "Datasheet" "" (at 270.51 27.94 0)
       (effects (font (size 1.27 1.27)) hide)
     )
@@
     )
   )
+  (symbol (lib_id "Connector:Conn_01x03_Pin") (at 262.89 24.13 270) (unit 1)
+    (in_bom yes) (on_board yes) (dnp no) (fields_autoplaced)
+    (property "Reference" "J1" (at 262.89 19.05 90)
+      (effects (font (size 1.27 1.27)))
+    )
+    (property "Value" "VCC" (at 262.89 21.59 90)
+      (effects (font (size 1.27 1.27)))
+    )
+    (property "Footprint" "" (at 262.89 24.13 0)
+      (effects (font (size 1.27 1.27)) hide)
+    )
+    (property "Datasheet" "~" (at 262.89 24.13 0)
+      (effects (font (size 1.27 1.27)) hide)
+    )
+    (pin "1")
+    (pin "2")
+    (pin "3")
+    (instances
+      (project "ExperimentNAND"
+        (path "/841976ed-b9e7-44ec-9bf3-24ace7a743f0"
+          (reference "J1") (unit 1)
+        )
+      )
+    )
+  )
   (symbol (lib_id "74xx:74HC00") (at 36.83 179.07 0) (unit 1)
     (in_bom yes) (on_board yes) (dnp no) (fields_autoplaced)
@@
         )
       )
+    )
+  )
+  (symbol (lib_id "power:+3.3V") (at 255.27 27.94 0) (unit 1)
+    (in_bom yes) (on_board yes) (dnp no) (fields_autoplaced)
+    (property "Reference" "#PWR017" (at 255.27 31.75 0)
+      (effects (font (size 1.27 1.27)) hide)
+    )
+    (property "Value" "+3.3V" (at 255.27 22.86 0)
+      (effects (font (size 1.27 1.27)))
+    )
+    (property "Footprint" "" (at 255.27 27.94 0)
+      (effects (font (size 1.27 1.27)) hide)
+    )
+    (property "Datasheet" "" (at 255.27 27.94 0)
+      (effects (font (size 1.27 1.27)) hide)
+    )
+    (pin "1")
+    (instances
+      (project "ExperimentNAND"
+        (path "/841976ed-b9e7-44ec-9bf3-24ace7a743f0"
+          (reference "#PWR017") (unit 1)
+        )
+      )
