File: KiCAD/Speaker/Speaker.kicad_sch (KiCad schematic)
At the start: 22 parts, among them J1 8P8C, Q1 2N3055, U1 MCP4801, U2 LM4562

Commit message: changed schemtatic to version 2.1
Parts:
- removed Q1: 2N3055, Package_TO_SOT_THT:TO-3, symbol Transistor_BJT:2N3055
- added C2, C4: 1uF, Capacitor_THT:CP_Radial_D5.0mm_P2.50mm, symbol Device:C_Polarized
- added C3: 10n, Capacitor_SMD:C_1206_3216Metric_Pad1.33x1.80mm_HandSolder, symbol Device:C
- added JP2: PERM ON, Jumper:SolderJumper-2_P1.3mm_Open_Pad1.0x1.5mm, symbol Jumper:SolderJumper_2_Open
- added R5: 10k, Resistor_SMD:R_0805_2012Metric_Pad1.20x1.40mm_HandSolder, symbol Device:R
- added TP4: TestPoint Signal, TestPoint:TestPoint_Loop_D2.54mm_Drill1.5mm_Beaded, symbol Connector:TestPoint
- added U3: LM4871, Package_SO:SOIC-8_5.23x5.23mm_P1.27mm, symbol LM4871:LM4871
- JP1: value SJ_R_Trim -> REMOTE SHTDWN
- R6: value 4.7k -> 10k
- renumbered R2 to R1, R3 to R2, R4 to R3, R1 to R4, R5 to R7, TP5 to TP1, TP4 to TP2, TP1 to TP3, TP2 to TP5, TP3 to TP6, U2 to U1, U1 to U2
Connections:
- net +5V: now also C3.1, C4.1, U3.6 (VDD)
- net GND: now also R7.1, C2.2, C3.2, C4.2, JP2.1 (A), U3.7 (GND); no longer LS1.2, R6.2, U1.5 (+), U1.6 (-)
- net at R7.3, TP5.1, U1.1: now also U1.2 (-); no longer JP1.2 (B)
- net at LS1.1, TP6.1: now also R6.2, U3.5 (V01)
- net at U1.7: now also U1.6 (-), R5.2, TP4.1
- net MISO renamed SHUTDOWN
- net SHUTDOWN: now also JP1.1 (A)
- new net: LS1.2, U3.8 (V02)
- new net: JP1.2 (B), JP2.2 (B), U3.1 (SHUTDOWN)
- new net: C2.1, U3.2 (BYPASS), U3.3 (+IN)
- new net: R5.1, R6.1, U3.4 (-IN)
- new net: R7.2, U1.5 (+)
- no-connect marks 3 -> 0
Other:
- moved on the sheet: C1, H1, H2, H3, H4, J1, LS1, R1, R2, R3, R4, R7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

Commit message: created PCB for version 2
Connections:
- net +3.3V is gone; now on net +5V: J1.2
- net +5V: now also U1.8 (V+)
- net CS: now also J1.3; no longer J1.4
- net GND: now also J1.7
- net MOSI: now also J1.5; no longer J1.6
- net SCK: now also J1.4; no longer J1.5
- net SHUTDOWN: now also J1.6; no longer J1.7
- removed net OPV_VCC: J1.3, U1.8 (V+)
Other:
- moved on the sheet: J1, R7, TP4, U1B
