File: KiCAD/Speaker/Speaker.kicad_pcb (KiCad board)
At the start: 2 copper layers, 100 x 50 mm, 22 parts, among them J1 8P8C, Q1 2N3055, U1 MCP4801, U2 LM4562

Commit message: created PCB for version 2
Parts:
- removed Q1: 2N3055, Package_TO_SOT_THT:TO-3
- removed the R4 at (152.5, 117.0)
- added C2: 1uF, Capacitor_THT:CP_Radial_D5.0mm_P2.50mm, F.Cu at (186.0, 89.0)
- added C3: 10n, Capacitor_SMD:C_1206_3216Metric_Pad1.33x1.80mm_HandSolder, F.Cu at (174.0, 115.0)
- added C4: 1uF, Capacitor_THT:CP_Radial_D5.0mm_P2.50mm, F.Cu at (186.0, 111.0)
- added JP2: PERM ON, Jumper:SolderJumper-2_P1.3mm_Open_Pad1.0x1.5mm, F.Cu at (176.3, 122.0)
- added R1: R, Resistor_SMD:R_0805_2012Metric_Pad1.20x1.40mm_HandSolder, F.Cu at (139.0, 117.0)
- added R7: Poti 10k, Potentiometer_THT:Potentiometer_Piher_PT-6-V_Vertical, F.Cu at (111.5, 118.5)
- added TP4: TestPoint Signal, TestPoint:TestPoint_Loop_D2.54mm_Drill1.5mm_Beaded, F.Cu at (164.0, 80.5)
- added U3: LM4871, Package_SO:SOIC-8_5.23x5.23mm_P1.27mm, F.Cu at (174.0, 107.0)
- JP1: value SJ_R_Trim -> REMOTE SHTDWN
- R5: value Poti 10k -> 10k; footprint Potentiometer_THT:Potentiometer_Piher_PT-6-V_Vertical -> Resistor_SMD:R_0805_2012Metric_Pad1.20x1.40mm_HandSolder
- R6: value 4.7k -> 10k
- moved R5 62.3 mm to (172.0, 96.0), turned to 90 degrees
- moved R6 37.8 mm to (166.0, 110.0), turned to -90 degrees
- moved JP1 34.5 mm to (162.8, 122.0), turned to 0 degrees
- moved TP6 14.0 mm to (178.5, 81.0)
- moved U1 10.7 mm to (156.8, 96.2), turned to -90 degrees
- moved R2 4.00 mm to (145.0, 117.0)
- moved R3 3.50 mm to (150.5, 117.0)
- renumbered R1 to R4, TP5 to TP1, TP4 to TP2, TP1 to TP3, TP2 to TP5, TP3 to TP6, U2 to U1, U1 to U2
Connections:
- J1 pad 2: +3.3V -> +5V
- J1 pad 3: /OPV_VCC -> /CS
- J1 pad 4: /CS -> /SCK
- J1 pad 5: /SCK -> /MOSI
- J1 pad 6: /MOSI -> /SHUTDOWN
- J1 pad 7: /MISO -> GND
- J1 pad 9: (no net) -> GND
- JP1 pad 1: Net-(JP1-A) -> /SHUTDOWN
- LS1 pad 1: Net-(Q1-E) -> Net-(U3-V01)
- LS1 pad 2: GND -> Net-(U3-V02)
- R5 pad 1: unconnected-(R5-Pad1) -> Net-(U3--IN)
- R5 pad 2: Net-(JP1-A) -> Net-(U1B--)
- R6 pad 1: Net-(JP1-A) -> Net-(U3--IN)
- R6 pad 2: GND -> Net-(U3-V01)
- TP5 pad 1: Net-(JP1-B) -> Net-(U1A--)
- TP6 pad 1: Net-(Q1-E) -> Net-(U3-V01)
- U1 pad 1: Net-(JP1-B) -> Net-(U1A--)
- U1 pad 2: Net-(JP1-A) -> Net-(U1A--)
- U1 pad 5: GND -> Net-(U1B-+)
- U1 pad 6: GND -> Net-(U1B--)
- U1 pad 7: unconnected-(U2-Pad7) -> Net-(U1B--)
- U1 pad 8: /OPV_VCC -> +5V
Routing:
- net /OPV_VCC: track 82.1 -> 0.00 mm
- net Net-(U1A--): track 0.00 -> 70.2 mm
- net Net-(U3-V01): track 0.00 -> 67.7 mm
- net Net-(JP1-A): track 63.1 -> 0.00 mm
- net /SHUTDOWN: track 0.00 -> 52.6 mm
- net GND: track 0.00 -> 45.3 mm
- net Net-(Q1-E): track 44.1 -> 0.00 mm
- net Net-(U1B--): track 0.00 -> 38.8 mm
- net Net-(U1B-+): track 0.00 -> 37.7 mm
- net Net-(JP1-B): track 112.8 -> 86.6 mm
- net Net-(U3-V02): track 0.00 -> 25.1 mm
- net +5V: track 118.1 -> 95.9 mm
- net Net-(U3-+IN): track 0.00 -> 20.4 mm
- net Net-(U3--IN): track 0.00 -> 14.9 mm
- net /CS: track 8.57 -> 11.1 mm
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Other:
- board text added: "TP Pre AMP"
- board text added: "Version 2.0"
- board text removed: "2N3055"
- board text removed: "Amp JP"
- board text removed: "Amplifier"
- board text removed: "DAC"
- board text removed: "Driver"
- board text removed: "Filter"
- board text removed: "SPI- Signal"
- board text removed: "Speaker"
- board text removed: "Version 1.0"
- board text removed: "Volume Amp"

Commit message: added plots + new audio controller
Other:
- board text added: "+"
- board text added: "-"
- board text added: "JLCJLCJLCJLC"
- board text added: "LM4871"
- board text added: "Volume Control"
