File: KiCAD/CabelAdapter/CabelAdapter.kicad_pcb (KiCad board)
At the start: 4 copper layers, 100 x 90 mm, 20 parts, among them J1 8P8C, J10 Conn_02x08_Odd_Even, J11 Conn_Coaxial, J12 Conn_01x04_Pin, J13 Conn_01x08_Pin, J14 Conn_Coaxial, J15 Screw_Terminal_01x08, J16 Conn_Coaxial, J17 Conn_01x04_Pin, J18 Conn_Coaxial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

Commit message: added mounting holes
Parts:
- added H1: MountingHole, MountingHole:MountingHole_3.2mm_M3, F.Cu at (85.0, 85.0)
- added H2: MountingHole, MountingHole:MountingHole_3.2mm_M3, F.Cu at (175.0, 85.0)
- added H3: MountingHole, MountingHole:MountingHole_3.2mm_M3, F.Cu at (175.0, 165.0)
- added H4: MountingHole, MountingHole:MountingHole_3.2mm_M3, F.Cu at (85.0, 165.0)
- moved J2 6.39 mm to (87.5, 93.2)
- moved J14 5.00 mm to (94.0, 150.8)
- moved J19 4.18 mm to (170.8, 156.8)
- moved J11 2.75 mm to (112.8, 150.8)
- moved J16 2.00 mm to (133.0, 150.8)
- moved J15 1.34 mm to (170.8, 110.2)
- moved J20 1.20 mm to (170.8, 142.3)
Routing:
- net /SIGNAL_2: track 355.0 -> 365.1 mm
- net /SIGNAL_1: track 360.8 -> 351.9 mm
- net GND: track 269.4 -> 263.3 mm
- net /SHUTDOWN: track 262.7 -> 256.6 mm
- net +5V: track 163.0 -> 156.9 mm
- net /SCK: track 250.0 -> 244.2 mm
- net /CS: track 199.0 -> 193.8 mm
- net /MOSI: track 287.4 -> 282.8 mm
- net /PIN_8: track 50.2 -> 47.4 mm
- net /PIN_1: track 50.6 -> 48.2 mm
- net /PIN_7: track 72.7 -> 70.5 mm
- net /PIN_6: track 71.6 -> 70.9 mm
- net /PIN_5: track 42.8 -> 42.3 mm
- net /PIN_2: track 72.4 -> 71.9 mm

Commit message: routed audio controller + added jlc string
Other:
- board text added: "JLCJLCJLCJLC"
Changed lines of the file:
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@@
     (effects (font (size 1 1) (thickness 0.15)) (justify bottom))
+  )
+  (gr_text "JLCJLCJLCJLC" (at 82.25 97.75) (layer "F.SilkS")
+    (effects (font (size 1 1) (thickness 0.15)) (justify left bottom))
   )
   (gr_text "SHDN" (at 143 87.25 90) (layer "F.SilkS")
