File: KiCAD/AudioController/AudioController.kicad_sch (KiCad schematic)
At the start: 39 parts, among them J1 8P8C, J10 CS_4_Measure, J11 CS_3_Measure, J12 CS_2_Measure, J13 CS_1_Measure, J14 CS_5_H, J15 CS_4_H, J16 CS_2_H, J17 CS_1_H, J18 MOSI_H, J19 SD_1_CTRL, J2 8P8C, J20 SCK_H, J21 SCK_Measure, J22 SD_2_CTRL, J23 SD_3_CTRL, J24 SD_4_CTRL, J25 SD_5_CTRL, J26 CS1_BR, J27 CS1_BR, J28 CS1_BR, J29 CS1_BR, J3 8P8C, J30 CS1_BR, J4 8P8C, J5 8P8C, J6 Power, J7 MOSI_Measure, J8 CS_3_H, J9 CS_5_Measure, U1 ESP32-DevKitC, U2 ESP32-DevKitC

Commit message: added audio controller pcb
Parts:
- added C1, C11, C13, C15, C3, C7, C9: 100nF, Capacitor_SMD:C_1206_3216Metric_Pad1.33x1.80mm_HandSolder, symbol Device:C
- added C10, C12, C14, C16, C2, C4, C8: 10uF, Capacitor_THT:CP_Radial_D5.0mm_P2.50mm, symbol Device:C_Polarized
- added D1, D2, D3, D4, D5, D6, D7, D8: LED, LED_THT:LED_D5.0mm, symbol Device:LED
- added H1, H2, H3, H4: MountingHole, MountingHole:MountingHole_3.2mm_M3, symbol Mechanical:MountingHole
- added R1, R10, R11, R12, R13, R14, R2, R3, R4, R5, R6, R7, R8, R9: 1k, Resistor_SMD:R_0805_2012Metric_Pad1.20x1.40mm_HandSolder, symbol Device:R
- added SW1, SW2, SW3, SW4, SW5, SW6: SW_Push, Button_Switch_THT:SW_PUSH_6mm, symbol Switch:SW_Push
- added TP1: SD_Card_MISO, TestPoint:TestPoint_Pad_D3.0mm, symbol Connector:TestPoint
- added TP10: TP_5V, TestPoint:TestPoint_Pad_D3.0mm, symbol Connector:TestPoint
- added TP2: SD_Card_MOSI, TestPoint:TestPoint_Pad_D3.0mm, symbol Connector:TestPoint
- added TP3: SD_Card_SCK, TestPoint:TestPoint_Pad_D3.0mm, symbol Connector:TestPoint
- added TP4: SD_Card_CS, TestPoint:TestPoint_Pad_D3.0mm, symbol Connector:TestPoint
- added TP5: DMA_MISO, TestPoint:TestPoint_Pad_D3.0mm, symbol Connector:TestPoint
- added TP6: DMA_MOSI, TestPoint:TestPoint_Pad_D3.0mm, symbol Connector:TestPoint
- added TP7: DMA_SCK, TestPoint:TestPoint_Pad_D3.0mm, symbol Connector:TestPoint
- added TP8: DMA_CS, TestPoint:TestPoint_Pad_D3.0mm, symbol Connector:TestPoint
- added TP9: CS_TP, TestPoint:TestPoint_Pad_D3.0mm, symbol Connector:TestPoint
- C5: renamed from C1; value 10nn -> 100nF; footprint (none) -> Capacitor_SMD:C_1206_3216Metric_Pad1.33x1.80mm_HandSolder
- C6: renamed from C2; footprint (none) -> Capacitor_THT:CP_Radial_D5.0mm_P2.50mm
- J1: renamed from J17; footprint (none) -> Connector_PinHeader_2.54mm:PinHeader_1x04_P2.54mm_Vertical
- J10: renamed from J23; footprint (none) -> Connector_PinHeader_2.54mm:PinHeader_1x03_P2.54mm_Vertical
- J11: renamed from J3; footprint (none) -> Library:RJ45_Amphenol_54602-x08_Horizontal_Custom
- J12: renamed from J11; footprint (none) -> Library:BNC_Connector
- J13: renamed from J15; footprint (none) -> Connector_PinHeader_2.54mm:PinHeader_1x04_P2.54mm_Vertical
- J14: renamed from J24; footprint (none) -> Connector_PinHeader_2.54mm:PinHeader_1x03_P2.54mm_Vertical
- J15: renamed from J4; footprint (none) -> Library:RJ45_Amphenol_54602-x08_Horizontal_Custom
- J16: renamed from J10; footprint (none) -> Library:BNC_Connector
- J17: renamed from J14; footprint (none) -> Connector_PinHeader_2.54mm:PinHeader_1x04_P2.54mm_Vertical
- J18: renamed from J25; footprint (none) -> Connector_PinHeader_2.54mm:PinHeader_1x03_P2.54mm_Vertical
- J19: renamed from J5; footprint (none) -> Library:RJ45_Amphenol_54602-x08_Horizontal_Custom
- J2: renamed from J19; footprint (none) -> Connector_PinHeader_2.54mm:PinHeader_1x03_P2.54mm_Vertical
- J20: renamed from J9; footprint (none) -> Library:BNC_Connector
- J21: renamed from J18; footprint (none) -> Connector_PinHeader_2.54mm:PinHeader_1x04_P2.54mm_Vertical
- J22: renamed from J7; footprint (none) -> Library:BNC_Connector
- J23: renamed from J20; footprint (none) -> Connector_PinHeader_2.54mm:PinHeader_1x04_P2.54mm_Vertical
- J24: renamed from J21; footprint (none) -> Library:BNC_Connector
- J25: renamed from J6; footprint (none) -> TerminalBlock_MetzConnect:TerminalBlock_MetzConnect_Type055_RT01502HDWU_1x02_P5.00mm_Horizontal
- J26, J27, J28, J29, J30: footprint (none) -> Connector_PinHeader_2.54mm:PinHeader_1x02_P2.54mm_Vertical
- J3: renamed from J1; footprint (none) -> Library:RJ45_Amphenol_54602-x08_Horizontal_Custom
- J4: renamed from J13; footprint (none) -> Library:BNC_Connector
- J5: renamed from J16; footprint (none) -> Connector_PinHeader_2.54mm:PinHeader_1x04_P2.54mm_Vertical
- J6: renamed from J22; footprint (none) -> Connector_PinHeader_2.54mm:PinHeader_1x03_P2.54mm_Vertical
- J7: renamed from J2; footprint (none) -> Library:RJ45_Amphenol_54602-x08_Horizontal_Custom
- J8: renamed from J12; footprint (none) -> Library:BNC_Connector
- J9: renamed from J8; footprint (none) -> Connector_PinHeader_2.54mm:PinHeader_1x04_P2.54mm_Vertical
- JP1: footprint (none) -> Jumper:SolderJumper-2_P1.3mm_Open_Pad1.0x1.5mm
- R15: renamed from R3; footprint (none) -> Resistor_SMD:R_0805_2012Metric_Pad1.20x1.40mm_HandSolder
- R16: renamed from R2; footprint (none) -> Resistor_SMD:R_0805_2012Metric_Pad1.20x1.40mm_HandSolder
- R17: renamed from R1; footprint (none) -> Resistor_SMD:R_0805_2012Metric_Pad1.20x1.40mm_HandSolder
- SD_Card_Reader1: footprint (none) -> Library:SD-Card_Adapter
Connections:
- net +5V: now also C1.1, C10.1, C11.1, C12.1, C13.1, C14.1, C15.1, C16.1, C2.1, C3.1, C4.1, C7.1, C8.1, C9.1, SW1.2, SW2.2, SW3.2, SW4.2, SW5.2, SW6.2, TP10.1
- net CS: now also TP9.1
- net DMA_CS: now also TP8.1
- net DMA_MISO: now also TP5.1
- net DMA_MOSI: now also TP6.1
- net DMA_SCK: now also TP7.1
- net GND: now also C1.2, C10.2, C11.2, C12.2, C13.2, C14.2, C15.2, C16.2, C2.2, C3.2, C4.2, C7.2, C8.2, C9.2, D1.1 (K), D2.1 (K), D3.1 (K), D4.1 (K), D5.1 (K), D6.1 (K), D7.1 (K), D8.1 (K), R1.2, R13.2, R14.2, R2.2, R3.2, R4.2
- net SD_CS: now also TP4.1
- net SD_MISO: now also TP1.1
- net SD_MOSI: now also TP2.1
- net SD_SCK: now also TP3.1
- net at U1.10 (DAC_2/ADC2_CH9/GPIO26): now also R6.1
- net at U1.11 (ADC2_CH7/GPIO27): now also R5.1
- net BTN_3: now reaches U1.3 (SENSOR_VP/GPIO36/ADC1_CH0)
- net BTN_3: now also R3.1, SW3.1
- net BTN_2: now reaches U1.36 (GPIO22)
- net BTN_2: now also R4.1, SW4.1
- net LED: now reaches U1.4 (SENSOR_VN/GPIO39/ADC1_CH3)
- net LED: now also R8.1
- net BTN_1: now reaches U1.5 (VDET_1/GPIO34/ADC1_CH6)
- net BTN_1: now also R2.1, SW2.1
- net BTN_4: now reaches U1.6 (VDET_2/GPIO35/ADC1_CH7)
- net BTN_4: now also R1.1, SW1.1
- net at U1.9 (DAC_1/ADC2_CH8/GPIO25): now also R7.1
- net BTN_5: now reaches U2.24 (ADC2_CH2/GPIO2)
- net BTN_5: now also R13.1, SW5.1
- net SD_ESP32: now reaches U2.26 (ADC2_CH0/GPIO4)
- net SD_ESP32: now also J10.1 (Pin_1), J14.1 (Pin_1), J18.1 (Pin_1), J2.1 (Pin_1), J6.1 (Pin_1)
- net at U2.3 (SENSOR_VP/GPIO36/ADC1_CH0): now also R11.1
- net at U2.4 (SENSOR_VN/GPIO39/ADC1_CH3): now also R9.1
- net at U2.5 (VDET_1/GPIO34/ADC1_CH6): now also R12.1
- net at U2.6 (VDET_2/GPIO35/ADC1_CH7): now also R10.1
- net BTN_6: now reaches U2.7 (32K_XP/GPIO32/ADC1_CH4)
- net BTN_6: now also R14.1, SW6.1
- net SD_1_Pin: no longer names the net of U2.20 (SD_CLK/GPIO6)
- net SD_1_Pin: no longer J2.1 (Pin_1)
- net SD_2_Pin: no longer names the net of U2.21 (SD_DATA0/GPIO7)
- net SD_2_Pin: no longer J6.1 (Pin_1)
- net SD_3_Pin: no longer names the net of U2.22 (SD_DATA1/GPIO8)
- net SD_3_Pin: no longer J10.1 (Pin_1)
- net SD_4_Pin: no longer names the net of U2.16 (SD_DATA2/GPIO9)
- net SD_4_Pin: no longer J14.1 (Pin_1)
- net SD_5_Pin: no longer names the net of U2.17 (SD_DATA3/GPIO10)
- net SD_5_Pin: no longer J18.1 (Pin_1)
- new net: D2.2 (A), R6.2
- new net: D5.2 (A), R9.2
- new net: D6.2 (A), R10.2
- new net: D7.2 (A), R11.2
- new net: D8.2 (A), R12.2
- new net: D1.2 (A), R5.2
- new net: D3.2 (A), R7.2
- new net: D4.2 (A), R8.2
- no-connect marks 43 -> 33
Other:
- title: (none) -> Audio Controller
- moved on the sheet: C5, C6, J10, J11, J12, J13, J14, J15, J16, J17, J18, J19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

Commit message: fixed pin assignment sd-card
Connections:
- net +5V: now also SD_Card_Reader1.2 (VCC); no longer SD_Card_Reader1.1 (GND)
- net GND: now also SD_Card_Reader1.1 (GND); no longer SD_Card_Reader1.2 (VCC)
Changed lines of the file:
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@@
     )
   )
-  (symbol (lib_id "power:+5V") (at 110.49 60.96 0) (mirror y) (unit 1)
-    (in_bom yes) (on_board yes) (dnp no) (fields_autoplaced)
-    (property "Reference" "#PWR034" (at 110.49 64.77 0)
-      (effects (font (size 1.27 1.27)) hide)
-    )
-    (property "Value" "+5V" (at 110.49 55.88 0)
-      (effects (font (size 1.27 1.27)))
-    )
-    (property "Footprint" "" (at 110.49 60.96 0)
-      (effects (font (size 1.27 1.27)) hide)
-    )
-    (property "Datasheet" "" (at 110.49 60.96 0)
+  (symbol (lib_id "power:+5V") (at 115.57 60.96 0) (mirror y) (unit 1)
+    (in_bom yes) (on_board yes) (dnp no) (fields_autoplaced)
+    (property "Reference" "#PWR034" (at 115.57 64.77 0)
+      (effects (font (size 1.27 1.27)) hide)
+    )
+    (property "Value" "+5V" (at 115.57 55.88 0)
+      (effects (font (size 1.27 1.27)))
+    )
+    (property "Footprint" "" (at 115.57 60.96 0)
+      (effects (font (size 1.27 1.27)) hide)
+    )
+    (property "Datasheet" "" (at 115.57 60.96 0)
       (effects (font (size 1.27 1.27)) hide)
     )
@@
     )
   )
-  (symbol (lib_id "power:GND") (at 115.57 60.96 0) (mirror x) (unit 1)
-    (in_bom yes) (on_board yes) (dnp no) (fields_autoplaced)
-    (property "Reference" "#PWR036" (at 115.57 54.61 0)
-      (effects (font (size 1.27 1.27)) hide)
-    )
-    (property "Value" "GND" (at 115.57 55.88 0)
-      (effects (font (size 1.27 1.27)))
-    )
-    (property "Footprint" "" (at 115.57 60.96 0)
-      (effects (font (size 1.27 1.27)) hide)
-    )
-    (property "Datasheet" "" (at 115.57 60.96 0)
-      (effects (font (size 1.27 1.27)) hide)
-    )
+  (symbol (lib_id "power:GND") (at 110.49 60.96 0) (mirror x) (unit 1)
+    (in_bom yes) (on_board yes) (dnp no) (fields_autoplaced)
+    (property "Reference" "#PWR036" (at 110.49 54.61 0)
+      (effects (font (size 1.27 1.27)) hide)
+    )
+    (property "Value" "GND" (at 110.49 55.88 0)
+      (effects (font (size 1.27 1.27)))
+    )
+    (property "Footprint" "" (at 110.49 60.96 0)
+      (effects (font (size 1.27 1.27)) hide)
+    )
+    (property "Datasheet" "" (at 110.49 60.96 0)
+      (effects (font (size 1.27 1.27)) hide)
+    )

Commit message: fixed pin assignments
Parts:
- removed D8: LED, LED_THT:LED_D5.0mm, symbol Device:LED
- removed JP1: SolderJumper_2_Open, Jumper:SolderJumper-2_P1.3mm_Open_Pad1.0x1.5mm, symbol Jumper:SolderJumper_2_Open
- added J31, J32, J33: Power Bridge, symbol Connector:Conn_01x02_Pin
- added R18: 1k, Resistor_SMD:R_0805_2012Metric_Pad1.20x1.40mm_HandSolder, symbol Device:R
- added SW7, SW8: SW_Push, Button_Switch_THT:SW_PUSH_6mm, symbol Switch:SW_Push
Connections:
- net +5V: now also J31.1 (Pin_1), J32.1 (Pin_1), SW7.2, SW8.2; no longer U1.19 (5V), U2.19 (5V)
- net BTN_2: now also U1.4 (SENSOR_VN/GPIO39/ADC1_CH3); no longer U1.36 (GPIO22)
- net BTN_5: now also U2.5 (VDET_1/GPIO34/ADC1_CH6); no longer U2.24 (ADC2_CH2/GPIO2)
- net BTN_6: now also U2.6 (VDET_2/GPIO35/ADC1_CH7); no longer U2.7 (32K_XP/GPIO32/ADC1_CH4)
- net DMA_CS: no longer TP8.1
- net GND: now also R12.2, R18.2
- net LED: now also R10.1, U2.24 (ADC2_CH2/GPIO2); no longer R8.1, U1.4 (SENSOR_VN/GPIO39/ADC1_CH3)
- net MOSI: now also J33.1 (Pin_1)
- net MOSI_ESP: now also J33.2 (Pin_2)
- net at R11.1: now also U2.7 (32K_XP/GPIO32/ADC1_CH4); no longer U2.3 (SENSOR_VP/GPIO36/ADC1_CH0)
- net at R9.1: now also U2.8 (32K_XN/GPIO33/ADC1_CH5); no longer U2.4 (SENSOR_VN/GPIO39/ADC1_CH3)
- net BTN_7: now reaches R12.1
- net BTN_7: now also U2.3 (SENSOR_VP/GPIO36/ADC1_CH0), SW7.1; no longer U2.5 (VDET_1/GPIO34/ADC1_CH6)
- new net: J32.2 (Pin_2), U1.19 (5V)
- new net: R8.1, U1.36 (GPIO22)
- new net: J31.2 (Pin_2), U2.19 (5V)
- new net BTN_8: R18.1, SW8.1, U2.4 (SENSOR_VN/GPIO39/ADC1_CH3)
- no-connect marks 33 -> 32
Other:
- moved on the sheet: TP5, TP6, TP7

Commit message: changed CS selector
Parts:
- removed D6: LED, LED_THT:LED_D5.0mm, symbol Device:LED
- removed J26, J27, J28, J29, J30: CS1_BR, Connector_PinHeader_2.54mm:PinHeader_1x02_P2.54mm_Vertical, symbol Connector:Conn_01x02_Pin
- removed R10, R12, R18: 1k, Resistor_SMD:R_0805_2012Metric_Pad1.20x1.40mm_HandSolder, symbol Device:R
- removed SW7, SW8: SW_Push, Button_Switch_THT:SW_PUSH_6mm, symbol Switch:SW_Push
- added J26: CS1_CTRL, Connector_PinHeader_2.54mm:PinHeader_1x03_P2.54mm_Vertical, symbol Connector:Conn_01x03_Pin
- added J27: CS2_CTRL, Connector_PinHeader_2.54mm:PinHeader_1x03_P2.54mm_Vertical, symbol Connector:Conn_01x03_Pin
- added J28: CS3_CTRL, Connector_PinHeader_2.54mm:PinHeader_1x03_P2.54mm_Vertical, symbol Connector:Conn_01x03_Pin
- added J29: CS4_CTRL, Connector_PinHeader_2.54mm:PinHeader_1x03_P2.54mm_Vertical, symbol Connector:Conn_01x03_Pin
- added J30: CS5_CTRL, Connector_PinHeader_2.54mm:PinHeader_1x03_P2.54mm_Vertical, symbol Connector:Conn_01x03_Pin
- added J34: Pin Bridge, symbol Connector_Generic:Conn_02x02_Odd_Even
Connections:
- net LED is gone; now on net COM_C: U2.24 (ADC2_CH2/GPIO2)
- net BTN_2: now also U1.33 (GPIO21); no longer U1.4 (SENSOR_VN/GPIO39/ADC1_CH3)
- net BTN_3: now also U1.26 (ADC2_CH0/GPIO4); no longer U1.3 (SENSOR_VP/GPIO36/ADC1_CH0)
- net CS: now also J26.3 (Pin_3), J27.3 (Pin_3), J28.3 (Pin_3), J29.3 (Pin_3), J30.3 (Pin_3)
- net CS_1: now also J26.2 (Pin_2); no longer U2.33 (GPIO21)
- net CS_2: now also J27.2 (Pin_2); no longer U2.36 (GPIO22)
- net CS_3: now also J28.2 (Pin_2); no longer U2.9 (DAC_1/ADC2_CH8/GPIO25)
- net CS_4: now also J29.2 (Pin_2); no longer U2.10 (DAC_2/ADC2_CH9/GPIO26)
- net CS_5: now also J30.2 (Pin_2); no longer U2.11 (ADC2_CH7/GPIO27)
- net DMA_CS: now also TP8.1
- net COM_C: now reaches U1.24 (ADC2_CH2/GPIO2)
- net at U1.7 (32K_XP/GPIO32/ADC1_CH4): now also J34.1 (Pin_1)
- net at U1.8 (32K_XN/GPIO33/ADC1_CH5): now also J34.3 (Pin_3)
- net BTN_7: no longer names the net of U2.3 (SENSOR_VP/GPIO36/ADC1_CH0)
- net BTN_7: now also J34.2 (Pin_2)
- net BTN_8: no longer names the net of U2.4 (SENSOR_VN/GPIO39/ADC1_CH3)
- net BTN_8: now also J34.4 (Pin_4)
- new net: J28.1 (Pin_1), U2.9 (DAC_1/ADC2_CH8/GPIO25)
- new net: J27.1 (Pin_1), U2.36 (GPIO22)
- new net: J30.1 (Pin_1), U2.11 (ADC2_CH7/GPIO27)
- new net: J26.1 (Pin_1), U2.33 (GPIO21)
- new net: J29.1 (Pin_1), U2.10 (DAC_2/ADC2_CH9/GPIO26)
- no-connect marks 32 -> 29
Other:
- moved on the sheet: C3, C4, D1, D2, D3, D4, D5, D7, H1, H2, H3, H4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

Commit message: routed audio controller + added jlc string
Parts:
- removed D1, D2, D3, D4, D5, D7: LED, LED_THT:LED_D5.0mm, symbol Device:LED
- removed R11, R13, R14, R9: 1k, Resistor_SMD:R_0805_2012Metric_Pad1.20x1.40mm_HandSolder, symbol Device:R
- removed SW5, SW6: SW_Push, Button_Switch_THT:SW_PUSH_6mm, symbol Switch:SW_Push
- added C17, C18, C19: 100nF, Capacitor_SMD:C_1206_3216Metric_Pad1.33x1.80mm_HandSolder, symbol Device:C
- added D10, D11, D12, D13, D14, D15, D17, D19, D4, D6, D8, D9: WS2812B, LED_SMD:LED_WS2812B_PLCC4_5.0x5.0mm_P3.2mm, symbol LED:WS2812B
- added JP1: PWR_JMP, Jumper:SolderJumper-2_P1.3mm_Open_Pad1.0x1.5mm, symbol Jumper:SolderJumper_2_Open
- added JP2: SJ_C_C2, Jumper:SolderJumper-2_P1.3mm_Open_Pad1.0x1.5mm, symbol Jumper:SolderJumper_2_Open
- added JP3: SJ_C_C3, Jumper:SolderJumper-2_P1.3mm_Open_Pad1.0x1.5mm, symbol Jumper:SolderJumper_2_Open
- added JP4: SJ_C_C4, Jumper:SolderJumper-2_P1.3mm_Open_Pad1.0x1.5mm, symbol Jumper:SolderJumper_2_Open
- added JP5: SJ_C_C1, Jumper:SolderJumper-2_P1.3mm_Open_Pad1.0x1.5mm, symbol Jumper:SolderJumper_2_Open
- added RV1: R_MOSI, Potentiometer_THT:Potentiometer_Piher_PT-6-V_Vertical, symbol Device:R_Potentiometer
- added SW7: POWER_SW, Library:Goobay10020, symbol Switch:SW_SPDT
- added TP11: COM_C2, TestPoint:TestPoint_Pad_D3.0mm, symbol Connector:TestPoint
- added TP12: COM_C3, TestPoint:TestPoint_Pad_D3.0mm, symbol Connector:TestPoint
- added TP13: COM_C4, TestPoint:TestPoint_Pad_D3.0mm, symbol Connector:TestPoint
- added TP14: COM_C1, TestPoint:TestPoint_Pad_D3.0mm, symbol Connector:TestPoint
- added TP15: LED_AP, TestPoint:TestPoint_Pad_D3.0mm, symbol Connector:TestPoint
- added TP16: LED_AB, TestPoint:TestPoint_Pad_D3.0mm, symbol Connector:TestPoint
- J31, J32: footprint (none) -> Connector_PinHeader_2.54mm:PinHeader_1x02_P2.54mm_Vertical
- J33: value Power Bridge -> MOSI Bridge; footprint (none) -> Connector_PinHeader_2.54mm:PinHeader_1x02_P2.54mm_Vertical
- J34: footprint (none) -> Connector_PinHeader_2.54mm:PinHeader_2x02_P2.54mm_Vertical
- R1, R2, R3, R4, R5, R6, R7, R8: value 1k -> 10k
- TP1: value SD_Card_MISO -> SD_MISO
- TP10: value TP_5V -> 5V
- TP2: value SD_Card_MOSI -> SD_MOSI
- TP3: value SD_Card_SCK -> SD_SCK
- TP4: value SD_Card_CS -> SD_CS
Connections:
- net +5V: now also C17.1, C18.1, C19.1, D10.1 (VDD), D11.1 (VDD), D12.1 (VDD), D13.1 (VDD), D14.1 (VDD), D15.1 (VDD), D17.1 (VDD), D19.1 (VDD), D4.1 (VDD), D6.1 (VDD), D8.1 (VDD), D9.1 (VDD), JP1.2 (B), SW7.1 (A); no longer C5.1, C6.1, J25.2 (Pin_2)
- net GND: now also R5.2, R6.2, R7.2, R8.2, C17.2, C18.2, C19.2, D10.3 (VSS), D11.3 (VSS), D12.3 (VSS), D13.3 (VSS), D14.3 (VSS), D15.3 (VSS), D17.3 (VSS), D19.3 (VSS), D4.3 (VSS), D6.3 (VSS), D8.3 (VSS), D9.3 (VSS), RV1.3
- net MOSI: now also RV1.2
- net MOSI_ESP: now also RV1.1
- net at R6.1, U1.10 (DAC_2/ADC2_CH9/GPIO26): now also JP3.2 (B)
- net at J27.1 (Pin_1): now also U2.33 (GPIO21); no longer U2.36 (GPIO22)
- net at U2.7 (32K_XP/GPIO32/ADC1_CH4): now also D4.4 (DIN), TP15.1
- net at R5.1, U1.11 (ADC2_CH7/GPIO27): now also JP4.2 (B)
- net at R8.1: now also U1.24 (ADC2_CH2/GPIO2), JP5.2 (B); no longer U1.36 (GPIO22)
- net at R7.1, U1.9 (DAC_1/ADC2_CH8/GPIO25): now also JP2.2 (B)
- net COM_C2: now reaches U2.8 (32K_XN/GPIO33/ADC1_CH5)
- net COM_C2: now also JP2.1 (A), TP11.1
- net at J26.1 (Pin_1): now also U2.36 (GPIO22); no longer U2.33 (GPIO21)
- net BTN_5 renamed COM_C3
- net COM_C3: now also JP3.1 (A), TP12.1
- net BTN_6 renamed COM_C4
- net COM_C4: now also JP4.1 (A), TP13.1
- net COM_C renamed COM_C1
- net COM_C1: now also JP5.1 (A), TP14.1; no longer U1.24 (ADC2_CH2/GPIO2)
- new net: C5.1, C6.1, J25.2 (Pin_2), JP1.1 (A), SW7.2 (B)
- new net: D17.2 (DOUT), D19.4 (DIN)
- new net: D13.2 (DOUT), D14.4 (DIN)
- new net: D10.2 (DOUT), D11.4 (DIN)
- new net: D10.4 (DIN), D9.2 (DOUT)
- new net: D8.2 (DOUT), D9.4 (DIN)
- new net: D6.2 (DOUT), D8.4 (DIN)
- new net: D6.4 (DIN), TP16.1, U1.36 (GPIO22)
- new net: D15.4 (DIN), D4.2 (DOUT)
- new net: D11.2 (DOUT), D12.4 (DIN)
- new net: D15.2 (DOUT), D17.4 (DIN)
- new net: D12.2 (DOUT), D13.4 (DIN)
- no-connect marks 29 -> 32
Other:
- moved on the sheet: C1, C10, C11, C12, C13, C14, C15, C16, C2, C3, C4, C5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
